File: PCB/pendulumControl.sch (EAGLE design)
At the start: 33 parts, among them IC1 PIC32MX340F512H, IC2 LT1963EST-3.3, Q1 8MHz

Commit message: Getting ready to remove some parts
Parts:
- removed IC2: LT1963EST-3.3, linear-technology:LT1963EST-3.3
- removed JP6: (no value), SparkFun-Connectors:M04PTH
- C9: value 10uF/6.3V -> 10uF/16V
Connections:
- new net VCC12V: C9.1, PAD1.P, R7.2
- net GND: no longer IC2G$1.GND, JP6.1
- net LIM_L: no longer JP6.2
- net LIM_R: no longer JP6.3
- net VCC3V3: no longer IC2G$1.OUT
- net VCC5V: no longer C9.1, IC2G$1.IN, JP6.4, PAD1.P, R7.2
Other:
- note removed: "Relay Output"
- note removed: "Voltage Regulator"
Changed lines of the file:
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@@
 <part name="C7" library="rcl" deviceset="C-US" device="C0805" value="2.2uF"/>
 <part name="C8" library="rcl" deviceset="C-US" device="C0805" value="2.2uF"/>
-<part name="JP6" library="SparkFun-Connectors" deviceset="M04" device="PTH"/>
-<part name="C9" library="rcl" deviceset="C-US" device="C0805" value="10uF/6.3V"/>
+<part name="C9" library="rcl" deviceset="C-US" device="C0805" value="10uF/16V"/>
 <part name="LED1" library="led" deviceset="LED" device="CHIP-LED0805" value="GRN"/>
 <part name="LED2" library="led" deviceset="LED" device="CHIP-LED0805" value="GRN"/>
 <part name="R6" library="rcl" deviceset="R-US_" device="R0805" value="60"/>
 <part name="R7" library="rcl" deviceset="R-US_" device="R0805" value="145"/>
-<part name="IC2" library="linear-technology" deviceset="LT1963EST" device="" technology="-3.3"/>
 <part name="Q1" library="crystal" deviceset="CRYSTAL" device="HC49S" value="8MHz"/>
 <part name="PAD1" library="wirepad" deviceset="3,81/1,4" device="" value="5V"/>
@@
 <wire x1="66.04" y1="-68.58" x2="99.06" y2="-68.58" width="0.1524" layer="97"/>
 <wire x1="99.06" y1="-68.58" x2="157.48" y2="-68.58" width="0.1524" layer="97"/>
-<wire x1="157.48" y1="-68.58" x2="195.58" y2="-68.58" width="0.1524" layer="97"/>
 <wire x1="-38.1" y1="-5.08" x2="-91.44" y2="-5.08" width="0.1524" layer="97"/>
 <wire x1="-91.44" y1="-5.08" x2="-111.76" y2="-5.08" width="0.1524" layer="97"/>
@@
 <wire x1="157.48" y1="-27.94" x2="157.48" y2="-68.58" width="0.1524" layer="97"/>
 <text x="142.24" y="-30.48" size="1.778" layer="97">Switch Input</text>
-<text x="160.02" y="-66.04" size="1.778" layer="97">Relay Output</text>
 <wire x1="157.48" y1="-27.94" x2="195.58" y2="-27.94" width="0.1524" layer="97"/>
-<wire x1="195.58" y1="-27.94" x2="195.58" y2="-68.58" width="0.1524" layer="97"/>
 <wire x1="-22.86" y1="111.76" x2="147.32" y2="111.76" width="0.1524" layer="97"/>
 <wire x1="147.32" y1="111.76" x2="147.32" y2="35.56" width="0.1524" layer="97"/>
@@
 <wire x1="-73.66" y1="66.04" x2="-22.86" y2="66.04" width="0.1524" layer="97"/>
 <text x="-38.1" y="35.56" size="1.778" layer="97">Status LEDs</text>
-<wire x1="147.32" y1="35.56" x2="195.58" y2="35.56" width="0.1524" layer="97"/>
-<wire x1="195.58" y1="35.56" x2="195.58" y2="-5.08" width="0.1524" layer="97"/>
 <text x="177.8" y="-25.4" size="1.778" layer="97">Power Input</text>
 <wire x1="195.58" y1="-5.08" x2="195.58" y2="-27.94" width="0.1524" layer="97"/>
 <wire x1="147.32" y1="-5.08" x2="195.58" y2="-5.08" width="0.1524" layer="97"/>
-<text x="170.18" y="-2.54" size="1.778" layer="97">Voltage Regulator</text>
 </plain>
 <instances>
@@
 <instance part="C7" gate="G$1" x="142.24" y="-45.72" rot="R90"/>
 <instance part="C8" gate="G$1" x="142.24" y="-55.88" rot="R90"/>
-<instance part="JP6" gate="G$1" x="165.1" y="-48.26"/>
 <instance part="C9" gate="G$1" x="-30.48" y="-53.34"/>
 <instance part="LED1" gate="G$1" x="-63.5" y="45.72"/>
@@
 <instance part="R6" gate="G$1" x="-63.5" y="55.88" rot="R90"/>
 <instance part="R7" gate="G$1" x="-50.8" y="55.88" rot="R90"/>
-<instance part="IC2" gate="G$1" x="167.64" y="20.32"/>
 <instance part="Q1" gate="G$1" x="-55.88" y="17.78"/>
 <instance part="PAD1" gate="1" x="152.4" y="-15.24"/>
@@
 </segment>
 <segment>
-<pinref part="JP6" gate="G$1" pin="1"/>
-<wire x1="170.18" y1="-50.8" x2="180.34" y2="-50.8" width="0.1524" layer="91"/>
-<label x="172.72" y="-50.8" size="1.778" layer="97"/>
-</segment>
-<segment>
 <pinref part="JP3" gate="G$1" pin="1"/>
 <wire x1="78.74" y1="-40.64" x2="86.36" y2="-40.64" width="0.1524" layer="91"/>
@@
 <label x="167.64" y="-17.78" size="1.778" layer="95"/>
 <pinref part="PAD2" gate="1" pin="P"/>
-</segment>
-<segment>
-<pinref part="IC2" gate="G$1" pin="GND"/>
-<wire x1="167.64" y1="15.24" x2="167.64" y2="10.16" width="0.1524" layer="91"/>
-<label x="167.64" y="10.16" size="1.778" layer="95"/>
 </segment>
 <segment>
@@
 </segment>
 <segment>
-<pinref part="IC2" gate="G$1" pin="OUT"/>
-<wire x1="177.8" y1="22.86" x2="187.96" y2="22.86" width="0.1524" layer="91"/>
-<label x="182.88" y="22.86" size="1.778" layer="95"/>
-</segment>
-<segment>
 <pinref part="IC1" gate="G$1" pin="AVDD"/>
 <wire x1="60.96" y1="-5.08" x2="60.96" y2="-15.24" width="0.1524" layer="91"/>
@@
 <junction x="116.84" y="-48.26"/>
 </segment>
-<segment>
-<pinref part="JP6" gate="G$1" pin="3"/>
-<wire x1="170.18" y1="-45.72" x2="180.34" y2="-45.72" width="0.1524" layer="91"/>
-<label x="172.72" y="-45.72" size="1.778" layer="97"/>
-</segment>
 </net>
 <net name="LIM_L" class="0">
@@
 <junction x="116.84" y="-50.8"/>
 </segment>
-<segment>
-<pinref part="JP6" gate="G$1" pin="2"/>
-<wire x1="170.18" y1="-48.26" x2="180.34" y2="-48.26" width="0.1524" layer="91"/>
-<label x="172.72" y="-48.26" size="1.778" layer="97"/>
-</segment>
 </net>
 <net name="VCC5V" class="0">
@@
 </segment>
 <segment>
-<pinref part="C9" gate="G$1" pin="1"/>
-<wire x1="-30.48" y1="-50.8" x2="-30.48" y2="-45.72" width="0.1524" layer="91"/>
-<label x="-30.48" y="-45.72" size="1.778" layer="97"/>
-</segment>
-<segment>
-<pinref part="JP6" gate="G$1" pin="4"/>
-<wire x1="170.18" y1="-43.18" x2="180.34" y2="-43.18" width="0.1524" layer="91"/>
-<label x="172.72" y="-43.18" size="1.778" layer="97"/>
-</segment>
-<segment>
 <pinref part="JP3" gate="G$1" pin="4"/>
 <wire x1="78.74" y1="-33.02" x2="86.36" y2="-33.02" width="0.1524" layer="91"/>
@@
 <wire x1="78.74" y1="-50.8" x2="86.36" y2="-50.8" width="0.1524" layer="91"/>
 <label x="81.28" y="-50.8" size="1.778" layer="97"/>
-</segment>
-<segment>
-<pinref part="R7" gate="G$1" pin="2"/>
-<wire x1="-50.8" y1="60.96" x2="-50.8" y2="63.5" width="0.1524" layer="91"/>
-<label x="-50.8" y="63.5" size="1.778" layer="97"/>
-</segment>
-<segment>
-<wire x1="154.94" y1="-15.24" x2="170.18" y2="-15.24" width="0.1524" layer="91"/>
-<label x="167.64" y="-15.24" size="1.778" layer="95"/>
-<pinref part="PAD1" gate="1" pin="P"/>
-</segment>
-<segment>
-<pinref part="IC2" gate="G$1" pin="IN"/>
-<wire x1="157.48" y1="22.86" x2="149.86" y2="22.86" width="0.1524" layer="91"/>
-<label x="149.86" y="22.86" size="1.778" layer="95"/>
 </segment>
 </net>
@@
 </segment>
 </net>
+<net name="VCC12V" class="0">
+<segment>
+<wire x1="154.94" y1="-15.24" x2="170.18" y2="-15.24" width="0.1524" layer="91"/>
+<label x="167.64" y="-15.24" size="1.778" layer="95"/>
+<pinref part="PAD1" gate="1" pin="P"/>
+</segment>
+<segment>
+<pinref part="C9" gate="G$1" pin="1"/>
+<wire x1="-30.48" y1="-50.8" x2="-30.48" y2="-45.72" width="0.1524" layer="91"/>
+<label x="-30.48" y="-45.72" size="1.778" layer="97"/>
+</segment>
+<segment>
+<pinref part="R7" gate="G$1" pin="2"/>
+<wire x1="-50.8" y1="60.96" x2="-50.8" y2="63.5" width="0.1524" layer="91"/>
+<label x="-50.8" y="63.5" size="1.778" layer="97"/>
+</segment>
+</net>
