File: PCB/pendulumControl.sch (EAGLE design)
At the start: 31 parts, among them IC1 PIC32MX340F512H, Q1 8MHz

Commit message: Updated the PCB
Parts:
- removed C7, C8: 2.2uF, rcl:C-USC0805
- removed JP3, JP4: (no value), SparkFun-Connectors:M04PTH
- removed JP5: (no value), SparkFun-Connectors:M03PTH
- removed R4, R5: 3.9k, rcl:R-US_R0805
- added ARM, MOTOR: (no value), SparkFun-Connectors:M03PTH
- added FAN: (no value), SparkFun-Connectors:M03POLAR
- added IC2: (no value), v-reg:78MXXS
- added LIMITS: (no value), SparkFun-Connectors:M02PTH
- R7: value 145 -> (none)
- renumbered JP1 to PROGRAMMING, JP2 to USB-UART, LED1 to 3.3V, LED2 to 12V, PAD1 to 24V, PAD2 to GND
Connections:
- removed net VCC5V: JP3.4, JP4.4, R4.2, R5.2
- new net VCC24V: 24V.P, IC2.IN
- net ARM_CHA: now also ARM.3; no longer JP3.3
- net ARM_CHB: now also ARM.2; no longer JP3.2
- net GND: now also ARM.1, FAN.1, IC2.GND, MOTOR.1; no longer C7.2, C8.2, JP3.1, JP4.1, JP5.1
- net LIM_L: now also LIMITS.2; no longer C8.1, JP5.3, R5.1
- net LIM_R: now also LIMITS.1; no longer C7.1, JP5.2, R4.1
- net M_CHA: now also MOTOR.3; no longer JP4.3
- net M_CHB: now also MOTOR.2; no longer JP4.2
- net VCC12V: now also FAN.2, IC2.OUT; no longer 24V.P
Other:
- note added: "Fan Output"
- note added: "Vreg"

Commit message: Added smoothing caps to the limit switches.
Parts:
- added C7, C8: 0.022uF, rcl:C-USC0805
Connections:
- net GND: now also C7.2, C8.2
- net LIM_L: now also C8.1
- net LIM_R: now also C7.1
Changed lines of the file:
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@@
 <part name="IC2" library="v-reg" deviceset="78MXXS" device=""/>
 <part name="FAN" library="SparkFun-Connectors" deviceset="M03" device="POLAR"/>
+<part name="C7" library="rcl" deviceset="C-US" device="C0805" value="0.022uF"/>
+<part name="C8" library="rcl" deviceset="C-US" device="C0805" value="0.022uF"/>
 </parts>
 <sheets>
@@
 <instance part="IC2" gate="A" x="177.8" y="-40.64"/>
 <instance part="FAN" gate="G$1" x="157.48" y="15.24"/>
+<instance part="C7" gate="G$1" x="121.92" y="-35.56" rot="R90"/>
+<instance part="C8" gate="G$1" x="121.92" y="-60.96" rot="R90"/>
 </instances>
 <busses>
@@
 <label x="172.72" y="12.7" size="1.778" layer="95"/>
 </segment>
+<segment>
+<pinref part="C7" gate="G$1" pin="2"/>
+<wire x1="127" y1="-35.56" x2="134.62" y2="-35.56" width="0.1524" layer="91"/>
+<label x="129.54" y="-35.56" size="1.778" layer="95"/>
+</segment>
+<segment>
+<pinref part="C8" gate="G$1" pin="2"/>
+<wire x1="127" y1="-60.96" x2="134.62" y2="-60.96" width="0.1524" layer="91"/>
+<label x="129.54" y="-60.96" size="1.778" layer="95"/>
+</segment>
 </net>
 <net name="VCC3V3" class="0">
@@
 <segment>
 <pinref part="LIMITS" gate="G$1" pin="1"/>
-<wire x1="114.3" y1="-48.26" x2="129.54" y2="-48.26" width="0.1524" layer="91"/>
+<wire x1="114.3" y1="-48.26" x2="116.84" y2="-48.26" width="0.1524" layer="91"/>
 <label x="129.54" y="-45.72" size="1.778" layer="95" rot="R180"/>
+<junction x="116.84" y="-48.26"/>
+<wire x1="116.84" y1="-48.26" x2="129.54" y2="-48.26" width="0.1524" layer="91"/>
+<wire x1="116.84" y1="-48.26" x2="116.84" y2="-35.56" width="0.1524" layer="91"/>
+<pinref part="C7" gate="G$1" pin="1"/>
+<wire x1="119.38" y1="-35.56" x2="116.84" y2="-35.56" width="0.1524" layer="91"/>
 </segment>
 </net>
@@
 <segment>
 <pinref part="LIMITS" gate="G$1" pin="2"/>
-<wire x1="114.3" y1="-50.8" x2="129.54" y2="-50.8" width="0.1524" layer="91"/>
+<wire x1="114.3" y1="-50.8" x2="116.84" y2="-50.8" width="0.1524" layer="91"/>
 <label x="129.54" y="-50.8" size="1.778" layer="95" rot="R180"/>
-</segment>
-</net>
+<junction x="116.84" y="-50.8"/>
+<wire x1="116.84" y1="-50.8" x2="129.54" y2="-50.8" width="0.1524" layer="91"/>
+<wire x1="116.84" y1="-50.8" x2="116.84" y2="-60.96" width="0.1524" layer="91"/>
+<pinref part="C8" gate="G$1" pin="1"/>
+<wire x1="116.84" y1="-60.96" x2="119.38" y2="-60.96" width="0.1524" layer="91"/>
+</segment>
+</net>

Commit message: Board is finalized and checked
Parts:
- added JP2: (no value), pinhead:PINHD-1X1
- LIMITS: device SparkFun-Connectors:M02PTH -> pinhead:PINHD-2X2
Connections:
- net GND: now also JP2.1
- net LIM_L: now also LIMITS.3, LIMITS.4; no longer LIMITS.2
- net LIM_R: now also LIMITS.2
Other:
- note removed: "Put Crystal Here"
Changed lines of the file:
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@@
 <part name="ARM" library="SparkFun-Connectors" deviceset="M03" device="PTH"/>
 <part name="MOTOR" library="SparkFun-Connectors" deviceset="M03" device="PTH"/>
-<part name="LIMITS" library="SparkFun-Connectors" deviceset="M02" device="PTH"/>
 <part name="C9" library="rcl" deviceset="C-US" device="C0805" value="10uF/16V"/>
 <part name="3.3V" library="led" deviceset="LED" device="CHIP-LED0805" value="GRN"/>
@@
 <part name="C7" library="rcl" deviceset="C-US" device="C0805" value="0.022uF"/>
 <part name="C8" library="rcl" deviceset="C-US" device="C0805" value="0.022uF"/>
+<part name="LIMITS" library="pinhead" deviceset="PINHD-2X2" device=""/>
+<part name="JP2" library="pinhead" deviceset="PINHD-1X1" device=""/>
 </parts>
 <sheets>
@@
 <wire x1="-73.66" y1="33.02" x2="-22.86" y2="33.02" width="0.1524" layer="97"/>
 <text x="-35.56" y="-2.54" size="1.778" layer="97">Oscillator</text>
-<text x="-101.6" y="38.1" size="1.778" layer="97">Put Crystal
-Here</text>
 <wire x1="27.94" y1="-27.94" x2="66.04" y2="-27.94" width="0.1524" layer="97"/>
 <wire x1="66.04" y1="-27.94" x2="66.04" y2="-68.58" width="0.1524" layer="97"/>
@@
 <instance part="ARM" gate="G$1" x="73.66" y="-38.1"/>
 <instance part="MOTOR" gate="G$1" x="73.66" y="-55.88"/>
-<instance part="LIMITS" gate="G$1" x="106.68" y="-48.26" rot="MR180"/>
 <instance part="C9" gate="G$1" x="-30.48" y="-53.34"/>
 <instance part="3.3V" gate="G$1" x="-63.5" y="45.72"/>
@@
 <instance part="C7" gate="G$1" x="121.92" y="-35.56" rot="R90"/>
 <instance part="C8" gate="G$1" x="121.92" y="-60.96" rot="R90"/>
+<instance part="LIMITS" gate="A" x="111.76" y="-50.8"/>
+<instance part="JP2" gate="G$1" x="149.86" y="-38.1" rot="R90"/>
 </instances>
 <busses>
@@
 <label x="129.54" y="-60.96" size="1.778" layer="95"/>
 </segment>
+<segment>
+<pinref part="JP2" gate="G$1" pin="1"/>
+<wire x1="149.86" y1="-40.64" x2="149.86" y2="-50.8" width="0.1524" layer="91"/>
+<label x="149.86" y="-50.8" size="1.778" layer="95" rot="R90"/>
+</segment>
 </net>
 <net name="VCC3V3" class="0">
@@
 </segment>
 <segment>
-<pinref part="LIMITS" gate="G$1" pin="1"/>
 <wire x1="114.3" y1="-48.26" x2="116.84" y2="-48.26" width="0.1524" layer="91"/>
 <label x="129.54" y="-45.72" size="1.778" layer="95" rot="R180"/>
@@
 <pinref part="C7" gate="G$1" pin="1"/>
 <wire x1="119.38" y1="-35.56" x2="116.84" y2="-35.56" width="0.1524" layer="91"/>
+<pinref part="LIMITS" gate="A" pin="2"/>
+<pinref part="LIMITS" gate="A" pin="1"/>
+<wire x1="106.68" y1="-48.26" x2="114.3" y2="-48.26" width="0.1524" layer="91"/>
+<junction x="114.3" y="-48.26"/>
 </segment>
 </net>
@@
 </segment>
 <segment>
-<pinref part="LIMITS" gate="G$1" pin="2"/>
 <wire x1="114.3" y1="-50.8" x2="116.84" y2="-50.8" width="0.1524" layer="91"/>
 <label x="129.54" y="-50.8" size="1.778" layer="95" rot="R180"/>
@@
 <pinref part="C8" gate="G$1" pin="1"/>
 <wire x1="116.84" y1="-60.96" x2="119.38" y2="-60.96" width="0.1524" layer="91"/>
+<pinref part="LIMITS" gate="A" pin="4"/>
+<pinref part="LIMITS" gate="A" pin="3"/>
+<wire x1="106.68" y1="-50.8" x2="114.3" y2="-50.8" width="0.1524" layer="91"/>
+<junction x="114.3" y="-50.8"/>
 </segment>
 </net>
@@
 <pinref part="FAN" gate="G$1" pin="2"/>
 <wire x1="165.1" y1="15.24" x2="177.8" y2="15.24" width="0.1524" layer="91"/>
+<label x="177.8" y="15.24" size="1.778" layer="95"/>
 </segment>
 </net>
@@
 </schematic>
 </drawing>
-<compatibility>
-<note version="6.3" minversion="6.2.2" severity="warning">
-Since Version 6.2.2 text objects can contain more than one line,
-which will not be processed correctly with this version.
-</note>
-</compatibility>
 </eagle>

Commit message: Added an excel parts list. Moved some silkscreen objects around
Parts:
- removed R8: 10k, resistor:R-US_R0805
- removed R9: 470, resistor:R-US_R0805
- added R4: 60, rcl:R-US_R0805
- added R5: 47, resistor:R-US_R0805
- C1: value 10uF/10V -> 100nF
- C10: value 0.1uF -> 0.022uF
- C11: value 100nF -> 0.022uF
- C2, C3: value 0.1uF -> 30pF; device resistor:C-USC0805 -> rcl:C-USC0805
- C4: value 0.1uF -> 10uF/16V; device resistor:C-USC0805 -> rcl:C-USC0805
- C5: value 30pF -> 0.1uF
- C6: value 30pF -> 0.1uF; device rcl:C-USC0805 -> resistor:C-USC0805
- C7, C8: value 0.022uF -> 0.1uF; device rcl:C-USC0805 -> resistor:C-USC0805
- C9: value 10uF/16V -> 10uF/10V
- R2: value 47 -> 680; device resistor:R-US_R0805 -> rcl:R-US_R0805
- R3: value 680 -> 10k; device rcl:R-US_R0805 -> resistor:R-US_R0805
- R6: value 60 -> 470; device rcl:R-US_R0805 -> resistor:R-US_R0805
- R7: value (none) -> 560
- renumbered 24V to PAD1, 3.3V to 3V3, GND to PAD2, JP2 to GRND
Connections:
- net LIM_L: now also C11.1; no longer C8.1
- net LIM_R: now also C10.1; no longer C7.1
- net MCLR: now also R6.2; no longer R9.2
- net N$1: now also R5.1; no longer R1.1
- net N$10: now also C9.1; no longer C1.1
- net N$2: now also R1.2; no longer R2.2
- net N$3: now also C2.1, R2.2; no longer C5.1, R3.2
- net N$4: now also R4.1; no longer R6.1
- net N$6: now also C1.1, R3.2, R6.1; no longer C11.1, R8.2, R9.1
- net OSC1: now also C3.1; no longer C6.1
- net OSC2: now also R2.1; no longer R3.1
- net P32_PGC: now also R1.1; no longer R2.1
- net P32_PGD: now also R5.2; no longer R1.2
- net VCC12V: now also C4.1; no longer C9.1
- net VCC3V3: now also C5.1, C6.1, C7.1, C8.1, R3.1, R4.2; no longer C10.1, C2.1, C3.1, C4.1, R6.2, R8.1
Other:
- moved on the sheet: C1, C10, C11, C2, C3, C4, C5, C6, C7, C8, C9, R1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
