File: PCB/pendulumControl.brd (EAGLE design)
At the start: 48 x 39.2 mm, 33 parts, among them IC1 PIC32MX340F512H, Q1 8MHz

Commit message: Board update
Parts:
- moved Q1 4.11 mm to (29.6, 10.3)
- moved C6 3.74 mm to (29.2, 15.3)
- moved C5 3.49 mm to (21.7, 11.9), turned to 0 degrees
Routing:
- net OSC2: track 19.8 -> 15.4 mm
- net OSC1: track 18.3 -> 15.7 mm
- net N$3: track 6.73 -> 8.51 mm
Changed lines of the file:
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@@
 <attribute name="VALUE" x="13.40904375" y="20.385428125" size="1.27" layer="27" rot="R180"/>
 </element>
-<element name="C5" library="rcl" package="C0805" value="30pF" x="25.114159375" y="11.301728125" rot="MR180"/>
-<element name="C6" library="rcl" package="C0805" value="30pF" x="29.313365625" y="11.53960625" smashed="yes" rot="MR0">
-<attribute name="NAME" x="30.6816125" y="9.1369375" size="1.27" layer="26" rot="MR0"/>
-<attribute name="VALUE" x="30.583365625" y="8.99960625" size="1.27" layer="28" rot="MR0"/>
+<element name="C5" library="rcl" package="C0805" value="30pF" x="21.675584375" y="11.92384375" rot="MR0"/>
+<element name="C6" library="rcl" package="C0805" value="30pF" x="29.22215625" y="15.280725" smashed="yes" rot="MR0">
+<attribute name="NAME" x="30.590403125" y="12.87805625" size="1.27" layer="26" rot="MR0"/>
+<attribute name="VALUE" x="30.49215625" y="12.740725" size="1.27" layer="28" rot="MR0"/>
 </element>
 <element name="C9" library="rcl" package="C0805" value="10uF/16V" x="39.37" y="26.67" smashed="yes" rot="MR90">
@@
 <attribute name="VALUE" x="9.194540625" y="21.111628125" size="1.27" layer="27" rot="R180"/>
 </element>
-<element name="Q1" library="crystal" package="HC49/S" value="8MHz" x="26.696553125" y="7.45105625">
-<attribute name="OC_NEWARK" value="unknown" x="26.696553125" y="7.45105625" size="1.778" layer="27" display="off"/>
-<attribute name="MPN" value="" x="26.696553125" y="7.45105625" size="1.778" layer="27" display="off"/>
-<attribute name="MF" value="" x="26.696553125" y="7.45105625" size="1.778" layer="27" display="off"/>
-<attribute name="OC_FARNELL" value="1667008" x="26.696553125" y="7.45105625" size="1.778" layer="27" display="off"/>
+<element name="Q1" library="crystal" package="HC49/S" value="8MHz" x="29.638003125" y="10.325328125">
+<attribute name="OC_NEWARK" value="unknown" x="29.638003125" y="10.325328125" size="1.778" layer="27" display="off"/>
+<attribute name="MPN" value="" x="29.638003125" y="10.325328125" size="1.778" layer="27" display="off"/>
+<attribute name="MF" value="" x="29.638003125" y="10.325328125" size="1.778" layer="27" display="off"/>
+<attribute name="OC_FARNELL" value="1667008" x="29.638003125" y="10.325328125" size="1.778" layer="27" display="off"/>
 </element>
 <element name="R1" library="resistor" package="R0805" value="47" x="10.16" y="13.97" smashed="yes" rot="MR180">
@@
 <contactref element="IC2" pad="GND"/>
 <contactref element="FAN" pad="1"/>
-<wire x1="2.83805" y1="20.49826875" x2="2.83805" y2="22.5069625" width="1.016" layer="1"/>
+<wire x1="2.83805" y1="20.49826875" x2="2.83805" y2="22.5069625" width="1.27" layer="1"/>
 <wire x1="2.83805" y1="22.5069625" x2="2.81919375" y2="22.52581875" width="1.016" layer="1"/>
-<wire x1="2.81919375" y1="22.52581875" x2="2.81919375" y2="26.45055" width="1.016" layer="1"/>
+<wire x1="2.81919375" y1="22.52581875" x2="2.81919375" y2="26.45055" width="1.27" layer="1"/>
 <wire x1="2.81919375" y1="26.45055" x2="3.610971875" y2="27.242328125" width="1.016" layer="1"/>
 <wire x1="18.0702875" y1="15.8902875" x2="18.07" y2="15.89" width="0.254" layer="1"/>
@@
 <contactref element="C5" pad="1"/>
 <contactref element="Q1" pad="1"/>
-<wire x1="24.283553125" y1="7.45105625" x2="24.164159375" y2="7.57045" width="0.254" layer="16"/>
-<wire x1="24.164159375" y1="7.57045" x2="24.164159375" y2="11.301728125" width="0.254" layer="16"/>
-<wire x1="24.164159375" y1="11.301728125" x2="22.61404375" y2="12.85184375" width="0.254" layer="16"/>
-<wire x1="22.61404375" y1="12.85184375" x2="22.61404375" y2="13.487040625" width="0.254" layer="16"/>
+<wire x1="22.625584375" y1="11.92384375" x2="24.87910625" y2="14.177365625" width="0.254" layer="16"/>
+<wire x1="24.87910625" y1="14.177365625" x2="25.733621875" y2="14.177365625" width="0.4064" layer="16"/>
+<wire x1="27.225003125" y1="10.325328125" x2="25.733621875" y2="11.816709375" width="0.254" layer="16"/>
+<wire x1="25.733621875" y1="11.816709375" x2="25.733621875" y2="14.177365625" width="0.254" layer="16"/>
 </signal>
 <signal name="OSC2">
 <contactref element="R3" pad="1"/>
 <contactref element="IC1" pad="40"/>
-<wire x1="22.61404375" y1="15.387040625" x2="24.598665625" y2="15.387040625" width="0.254" layer="16"/>
-<wire x1="24.598665625" y1="15.387040625" x2="25.811390625" y2="16.599765625" width="0.254" layer="16"/>
-<wire x1="25.811390625" y1="16.599765625" x2="28.7444375" y2="16.599765625" width="0.254" layer="16"/>
-<wire x1="28.7444375" y1="16.599765625" x2="29.331125" y2="17.186453125" width="0.254" layer="16"/>
-<via x="29.331125" y="17.186453125" extent="1-16" drill="0.5"/>
-<wire x1="29.331125" y1="17.186453125" x2="31.832871875" y2="17.186453125" width="0.254" layer="1"/>
-<wire x1="31.832871875" y1="17.186453125" x2="32.091703125" y2="17.445284375" width="0.254" layer="1"/>
-<wire x1="32.091703125" y1="17.445284375" x2="32.091703125" y2="20.51685625" width="0.254" layer="1"/>
-<wire x1="32.091703125" y1="20.51685625" x2="31.263825" y2="21.337803125" width="0.254" layer="1"/>
-<wire x1="31.263825" y1="21.337803125" x2="26.10790625" y2="21.344734375" width="0.254" layer="1"/>
-<wire x1="26.10790625" y1="21.344734375" x2="26.02" y2="21.34" width="0.254" layer="1"/>
+<wire x1="25.733621875" y1="16.077365625" x2="26.7893375" y2="17.13308125" width="0.254" layer="16"/>
+<wire x1="26.7893375" y1="17.13308125" x2="29.371625" y2="17.13308125" width="0.254" layer="16"/>
+<via x="29.371625" y="17.13308125" extent="1-16" drill="0.5"/>
+<wire x1="29.371625" y1="17.13308125" x2="30.954253125" y2="17.13308125" width="0.254" layer="1"/>
+<wire x1="30.954253125" y1="17.13308125" x2="31.83794375" y2="18.016771875" width="0.254" layer="1"/>
+<wire x1="31.83794375" y1="18.016771875" x2="31.83794375" y2="20.166703125" width="0.254" layer="1"/>
+<wire x1="31.83794375" y1="20.166703125" x2="30.63775625" y2="21.366890625" width="0.254" layer="1"/>
+<wire x1="30.63775625" y1="21.366890625" x2="26.046890625" y2="21.366890625" width="0.254" layer="1"/>
+<wire x1="26.046890625" y1="21.366890625" x2="26.02" y2="21.34" width="0.254" layer="1"/>
 </signal>
 <signal name="OSC1">
@@
 <contactref element="Q1" pad="2"/>
 <contactref element="IC1" pad="39"/>
-<wire x1="29.109553125" y1="7.45105625" x2="30.263365625" y2="8.60486875" width="0.254" layer="16"/>
-<wire x1="30.263365625" y1="8.60486875" x2="30.263365625" y2="11.53960625" width="0.254" layer="16"/>
-<wire x1="30.263365625" y1="11.53960625" x2="30.683809375" y2="11.96005" width="0.254" layer="16"/>
-<wire x1="30.683809375" y1="11.96005" x2="30.683809375" y2="18.26613125" width="0.254" layer="16"/>
 <via x="30.683809375" y="18.26613125" extent="1-16" drill="0.5"/>
 <wire x1="30.683809375" y1="18.26613125" x2="30.683809375" y2="20.088803125" width="0.254" layer="1"/>
@@
 <wire x1="29.938453125" y1="20.834159375" x2="26.025840625" y2="20.834159375" width="0.254" layer="1"/>
 <wire x1="26.025840625" y1="20.834159375" x2="26.02" y2="20.84" width="0.254" layer="1"/>
+<wire x1="30.17215625" y1="15.280725" x2="32.051003125" y2="13.401878125" width="0.254" layer="16"/>
+<wire x1="32.051003125" y1="13.401878125" x2="32.051003125" y2="10.325328125" width="0.254" layer="16"/>
+<wire x1="30.17215625" y1="15.280725" x2="30.683809375" y2="15.792378125" width="0.4064" layer="16"/>
+<wire x1="30.683809375" y1="15.792378125" x2="30.683809375" y2="18.26613125" width="0.254" layer="16"/>
 </signal>
 <signal name="RX">
@@
 <contactref element="IC1" pad="33"/>
 <wire x1="8.89" y1="6.35" x2="20.091203125" y2="17.551203125" width="0.254" layer="16"/>
-<wire x1="20.091203125" y1="17.551203125" x2="21.4956625" y2="17.6148" width="0.254" layer="16"/>
-<via x="21.4956625" y="17.6148" extent="1-16" drill="0.5"/>
-<wire x1="21.4956625" y1="17.6148" x2="25.731203125" y2="17.551203125" width="0.254" layer="1"/>
-<wire x1="25.731203125" y1="17.551203125" x2="26.02" y2="17.84" width="0.254" layer="1"/>
+<wire x1="20.091203125" y1="17.551203125" x2="21.251228125" y2="17.551203125" width="0.254" layer="16"/>
+<wire x1="21.251228125" y1="17.551203125" x2="21.251228125" y2="17.551528125" width="0.254" layer="16"/>
+<via x="21.251228125" y="17.551528125" extent="1-16" drill="0.5"/>
+<wire x1="21.251228125" y1="17.551528125" x2="25.731528125" y2="17.551528125" width="0.254" layer="1"/>
+<wire x1="25.731528125" y1="17.551528125" x2="26.02" y2="17.84" width="0.254" layer="1"/>
 </signal>
 <signal name="M_CHB">

Commit message: Fix conflicts
Parts:
- moved R3 1.23 mm to (23.5, 15.3), turned to 0 degrees
Routing:
- net GND: track 69.7 -> 77.8 mm, vias 8 -> 10
- net OSC2: track 15.4 -> 17.0 mm
Changed lines of the file:
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@@
 </element>
 <element name="R2" library="resistor" package="R0805" value="47" x="7.62" y="17.78" rot="MR0"/>
-<element name="R3" library="rcl" package="R0805" value="680" x="22.61404375" y="14.437040625" smashed="yes" rot="MR270">
-<attribute name="NAME" x="25.456715625" y="16.55345" size="1.27" layer="26" rot="MR270"/>
-<attribute name="VALUE" x="25.15404375" y="15.072040625" size="1.27" layer="28" rot="MR270"/>
+<element name="R3" library="rcl" package="R0805" value="680" x="23.523478125" y="15.2691375" smashed="yes" rot="MR0">
+<attribute name="NAME" x="25.6398875" y="12.426465625" size="1.27" layer="26" rot="MR0"/>
+<attribute name="VALUE" x="24.158478125" y="12.7291375" size="1.27" layer="28" rot="MR0"/>
 </element>
 <element name="R6" library="rcl" package="R0805" value="60" x="8.700559375" y="27.8262" rot="R90"/>
@@
 <wire x1="26.235784375" y1="15.484715625" x2="28.124090625" y2="17.373021875" width="0.254" layer="1"/>
 <wire x1="28.124090625" y1="17.373021875" x2="28.124090625" y2="17.93948125" width="0.254" layer="1"/>
-<wire x1="39.322409375" y1="15.114184375" x2="39.37" y2="3.81" width="0" layer="19" extent="16-16"/>
+<wire x1="39.322409375" y1="15.114184375" x2="37.85468125" y2="15.114184375" width="0.4064" layer="16"/>
+<wire x1="37.85468125" y1="15.114184375" x2="37.85468125" y2="15.121940625" width="0.4064" layer="16"/>
+<via x="37.85468125" y="15.121940625" extent="1-16" drill="0.5"/>
+<wire x1="37.85468125" y1="15.121940625" x2="37.85468125" y2="10.807309375" width="0.254" layer="1"/>
+<wire x1="37.85468125" y1="10.807309375" x2="37.896509375" y2="10.76548125" width="0.254" layer="1"/>
+<via x="37.896509375" y="10.76548125" extent="1-16" drill="0.5"/>
+<wire x1="37.896509375" y1="10.76548125" x2="37.56230625" y2="10.76548125" width="0.254" layer="16"/>
+<wire x1="37.56230625" y1="10.76548125" x2="37.269084375" y2="10.472259375" width="0.254" layer="16"/>
+<wire x1="20.725584375" y1="11.92384375" x2="20.44593125" y2="11.644190625" width="0.254" layer="16"/>
+<wire x1="20.44593125" y1="11.644190625" x2="19.358671875" y2="11.644190625" width="0.254" layer="16"/>
 </signal>
 <signal name="MCLR">
@@
 <contactref element="C5" pad="1"/>
 <contactref element="Q1" pad="1"/>
-<wire x1="22.625584375" y1="11.92384375" x2="24.87910625" y2="14.177365625" width="0.254" layer="16"/>
-<wire x1="24.87910625" y1="14.177365625" x2="25.733621875" y2="14.177365625" width="0.4064" layer="16"/>
-<wire x1="27.225003125" y1="10.325328125" x2="25.733621875" y2="11.816709375" width="0.254" layer="16"/>
-<wire x1="25.733621875" y1="11.816709375" x2="25.733621875" y2="14.177365625" width="0.254" layer="16"/>
+<wire x1="22.573478125" y1="15.2691375" x2="22.625584375" y2="15.21703125" width="0.254" layer="16"/>
+<wire x1="22.625584375" y1="15.21703125" x2="22.625584375" y2="11.92384375" width="0.254" layer="16"/>
+<wire x1="22.625584375" y1="11.92384375" x2="25.6264875" y2="11.92384375" width="0.254" layer="16"/>
+<wire x1="25.6264875" y1="11.92384375" x2="27.225003125" y2="10.325328125" width="0.254" layer="16"/>
 </signal>
 <signal name="OSC2">
 <contactref element="R3" pad="1"/>
 <contactref element="IC1" pad="40"/>
-<wire x1="25.733621875" y1="16.077365625" x2="26.7893375" y2="17.13308125" width="0.254" layer="16"/>
-<wire x1="26.7893375" y1="17.13308125" x2="29.371625" y2="17.13308125" width="0.254" layer="16"/>
-<via x="29.371625" y="17.13308125" extent="1-16" drill="0.5"/>
-<wire x1="29.371625" y1="17.13308125" x2="30.954253125" y2="17.13308125" width="0.254" layer="1"/>
+<wire x1="24.92539375" y1="15.2691375" x2="26.7893375" y2="17.13308125" width="0.254" layer="16"/>
+<wire x1="26.7893375" y1="17.13308125" x2="29.581621875" y2="17.1214125" width="0.254" layer="16"/>
+<via x="29.581621875" y="17.1214125" extent="1-16" drill="0.5"/>
+<wire x1="29.581621875" y1="17.1214125" x2="30.954253125" y2="17.13308125" width="0.254" layer="1"/>
 <wire x1="30.954253125" y1="17.13308125" x2="31.83794375" y2="18.016771875" width="0.254" layer="1"/>
 <wire x1="31.83794375" y1="18.016771875" x2="31.83794375" y2="20.166703125" width="0.254" layer="1"/>
@@
 <wire x1="30.63775625" y1="21.366890625" x2="26.046890625" y2="21.366890625" width="0.254" layer="1"/>
 <wire x1="26.046890625" y1="21.366890625" x2="26.02" y2="21.34" width="0.254" layer="1"/>
+<wire x1="24.92539375" y1="15.2691375" x2="24.473478125" y2="15.2691375" width="0.254" layer="16"/>
 </signal>
 <signal name="OSC1">

Commit message: Board is finalized and checked
Parts:
- added JP2: (no value), pinhead:1X01
- LIMITS: device SparkFun-Connectors:1X02 -> pinhead:2X02
- moved LIMITS 33.2 mm to (22.1, 36.0), turned to 90 degrees
- moved C8 29.4 mm to (15.8, 31.5), turned to 270 degrees
- moved C7 18.9 mm to (23.4, 31.2), turned to 270 degrees
Connections:
- net GND: now also JP2.1
- net LIM_L: now also LIMITS.3, LIMITS.4; no longer LIMITS.2
- net LIM_R: now also LIMITS.2
Routing:
- net LIM_R: track 37.7 -> 24.9 mm
- net LIM_L: track 35.2 -> 24.8 mm
- net GND: track 77.8 -> 71.6 mm, vias 10 -> 6
